File: Crowboard-Kicad/crowboard.kicad_pcb (KiCad board)
At the start: 2 copper layers, 73 parts, among them U1 Pico

Commit message: second
Parts:
- MX7: moved to B.Cu
- moved MX13 285.6 mm to (91.3, 70.6)
- moved D25 280.2 mm to (128.6, 80.2)
- moved MX35 266.0 mm to (167.5, 108.7)
- moved MX28 254.2 mm to (186.5, 89.7)
- moved MX26 246.2 mm to (148.4, 89.7)
- moved D12 219.6 mm to (104.3, 263.0)
- moved D18 219.6 mm to (83.5, 263.0)
- moved D21 219.6 mm to (114.7, 263.0)
- moved D29 219.6 mm to (52.3, 263.0)
- moved D3 219.6 mm to (93.9, 263.0)
- moved D32 219.6 mm to (125.1, 263.0)
- moved D33 219.6 mm to (73.1, 263.0)
- moved D6 219.6 mm to (62.7, 263.0)
- moved D1 219.6 mm to (83.5, 268.4)
- moved D10 219.6 mm to (114.7, 268.4)
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
Commit message: adjustments
Parts:
- MX7: moved to F.Cu
- moved D25 147.4 mm to (248.4, 165.9)
- moved D7 35.9 mm to (177.8, 182.6), turned to 90 degrees
- moved MX18 35.1 mm to (220.6, 61.9)
- moved MX28 35.1 mm to (220.6, 81.0)
- moved MX8 35.1 mm to (220.6, 42.9)
- moved MX10 34.4 mm to (258.7, 56.4)
- moved MX20 34.4 mm to (258.7, 75.4)
- moved MX30 34.4 mm to (258.7, 94.5)
- moved MX17 34.2 mm to (201.5, 66.7)
- moved MX27 34.2 mm to (201.5, 85.7)
- moved MX7 34.2 mm to (201.6, 47.6), turned to 0 degrees
- moved MX19 34.2 mm to (239.6, 66.7)
- moved MX29 34.2 mm to (239.6, 85.7)
- moved MX9 34.2 mm to (239.6, 47.6)
- moved MX16 34.1 mm to (182.5, 70.6)
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
Commit message: adjustments
Parts:
- moved D9 257.3 mm to (239.6, 56.4)
- moved D29 252.1 mm to (239.7, 94.5)
- moved D10 249.2 mm to (258.8, 65.1)
- moved D19 246.2 mm to (239.7, 75.4)
- moved D8 243.7 mm to (220.7, 51.6)
- moved D28 238.5 mm to (220.7, 89.7)
- moved D18 236.3 mm to (220.7, 70.6)
- moved D6 235.5 mm to (182.6, 60.3)
- moved D16 227.4 mm to (182.6, 79.4)
- moved D30 226.2 mm to (258.8, 103.2)
- moved D4 216.7 mm to (96.8, 56.4)
- moved D27 216.4 mm to (201.6, 94.5)
- moved D17 214.1 mm to (201.6, 75.4)
- moved D3 212.1 mm to (77.7, 51.6)
- moved D1 207.9 mm to (39.8, 65.1)
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Routing:
- net Net-(D35-Pad2): track 0.00 -> 41.4 mm
- net Net-(D36-Pad2): track 0.00 -> 38.4 mm
- net Net-(D34-Pad2): track 0.00 -> 29.1 mm

Commit message: finished
Parts:
- moved U1 249.2 mm to (149.1, 70.9)
- moved MX34 18.8 mm to (185.1, 135.2), turned to 45 degrees
- moved MX33 18.5 mm to (114.5, 135.3), turned to -45 degrees
- moved D30 14.6 mm to (265.9, 90.5), turned to 15 degrees
- moved D21 14.5 mm to (32.9, 90.4), turned to -15 degrees
- moved MX35 13.9 mm to (204.5, 121.8), turned to 35 degrees
- moved MX32 13.6 mm to (95.1, 121.9), turned to -35 degrees
- moved MX30 13.3 mm to (263.6, 82.1), turned to 15 degrees
- moved MX21 13.3 mm to (35.1, 82.0), turned to -15 degrees
- moved D34 13.0 mm to (193.6, 114.9), turned to 15 degrees
- moved D33 12.6 mm to (105.3, 114.7), turned to -15 degrees
- moved D35 12.4 mm to (192.8, 111.8), turned to 15 degrees
- moved MX1 12.4 mm to (45.0, 45.2), turned to -15 degrees
- moved D11 12.2 mm to (37.8, 72.0), turned to -15 degrees
- moved D20 12.2 mm to (261.0, 72.1), turned to 15 degrees
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Connections:
- U1 pad 10: unconnected-(U1-Pad10) -> COL1
- U1 pad 11: unconnected-(U1-Pad11) -> COL2
- U1 pad 12: unconnected-(U1-Pad12) -> COL3
- U1 pad 14: unconnected-(U1-Pad14) -> COL4
- U1 pad 19: unconnected-(U1-Pad19) -> ROW0
- U1 pad 20: unconnected-(U1-Pad20) -> ROW1
- U1 pad 21: unconnected-(U1-Pad21) -> ROW2
- U1 pad 22: unconnected-(U1-Pad22) -> ROW3
- U1 pad 27: unconnected-(U1-Pad27) -> COL5
- U1 pad 29: unconnected-(U1-Pad29) -> COL6
- U1 pad 30: unconnected-(U1-Pad30) -> COL7
- U1 pad 31: unconnected-(U1-Pad31) -> COL8
- U1 pad 32: unconnected-(U1-Pad32) -> COL9
- U1 pad 9: unconnected-(U1-Pad9) -> COL0
Routing:
- net ROW2: track 0.00 -> 433.1 mm, vias 0 -> 1
- net ROW0: track 0.00 -> 350.6 mm
- net ROW1: track 0.00 -> 349.8 mm, vias 0 -> 1
- net COL7: track 0.00 -> 193.9 mm
- net ROW3: track 0.00 -> 175.2 mm, vias 0 -> 2
- net COL0: track 0.00 -> 174.7 mm
- net COL2: track 0.00 -> 168.6 mm
- net COL9: track 0.00 -> 165.7 mm
- net COL1: track 0.00 -> 144.9 mm
- net COL3: track 0.00 -> 143.7 mm
- net COL8: track 0.00 -> 140.1 mm
- net COL6: track 0.00 -> 138.0 mm
- net COL4: track 0.00 -> 122.3 mm
- net COL5: track 0.00 -> 116.8 mm
- net Net-(D31-Pad2): track 0.00 -> 38.7 mm
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Other:
- board outline added: 251.9 x 118.8 mm

Commit message: final
Parts:
- added G***: LOGO, crow:crow50, F.Cu at (147.2, 111.1)
Other:
- board text added: "CROWBOARD"
