File: Crowboard-Kicad/crowboard.kicad_pcb (KiCad board)
At the start: 2 copper layers, 251.9 x 118.8 mm, 75 parts, among them U1 Pico

Commit message: fix routing
Connections:
- U1 pad 24: unconnected-(U1-Pad24) -> COL5
- U1 pad 25: unconnected-(U1-Pad25) -> COL6
- U1 pad 26: unconnected-(U1-Pad26) -> COL7
- U1 pad 27: COL5 -> COL8
- U1 pad 29: COL6 -> COL9
- U1 pad 30: COL7 -> unconnected-(U1-Pad30)
- U1 pad 31: COL8 -> unconnected-(U1-Pad31)
- U1 pad 32: COL9 -> unconnected-(U1-Pad32)
Routing:
- net COL9: track 165.7 -> 162.3 mm
- net COL5: track 116.8 -> 120.1 mm
- net COL6: track 138.0 -> 139.7 mm
- net COL8: track 140.1 -> 138.8 mm
