File: Crowboard-Kicad-rev2 MX/crowboard.kicad_pcb (KiCad board)
At the start: 2 copper layers, 251.9 x 118.8 mm, 79 parts, among them J1 Conn_01x05, J2 Conn_01x04, SW1 RotaryEncoder, SW2 RotaryEncoder, U1 Pico

Commit message: Crowboard Rev 2 MX
Parts:
- removed J1: Conn_01x05, other_parts:pimoroni
- added ec11-1: RotaryEncoder_Switch, Rotary_Encoder:RotaryEncoder_Alps_EC11E-Switch_Vertical_H20mm, F.Cu at (137.9, 117.6)
- added ec11-2: RotaryEncoder_Switch, Rotary_Encoder:RotaryEncoder_Alps_EC11E-Switch_Vertical_H20mm, F.Cu at (160.8, 112.5)
- BIG CROW: renamed from G***
- LITTLE CROW: renamed from G***
- MX1, MX10, MX11, MX12, MX13, MX14, MX15, MX16, MX17, MX18, MX19, MX2, MX20, MX21, MX22, MX23, MX24, MX25, MX26, MX27, MX28, MX29, MX3, MX30, MX31, MX32, MX33, MX34, MX35, MX36, MX4, MX5, MX6, MX7, MX8, MX9: footprint Keebio-Parts:Kailh-PG1350-1u-NoLED -> MX_Only:MXOnly-1U-NoLED
- moved ec12-1 14.4 mm to (132.3, 117.6), turned to 180 degrees
- moved ec12-2 0.19 mm to (166.5, 112.5)
- renumbered SW1 to ec12-1, SW2 to ec12-2, J2 to oled1
Connections:
- U1 pad 4: SDA -> unconnected-(U1-Pad4)
- U1 pad 5: SCL -> unconnected-(U1-Pad5)
Routing:
- net ROW2: track 433.1 -> 258.9 mm
- net COL8: track 138.8 -> 264.4 mm, vias 0 -> 1
- net SDA: track 88.3 -> 0.00 mm, vias 1 -> 0
- net ROW1: track 349.8 -> 264.1 mm
- net SCL: track 83.4 -> 0.00 mm, vias 1 -> 0
- net ROW0: track 350.6 -> 269.4 mm
- net GND1: track 71.6 -> 0.00 mm
- net COL1: track 144.9 -> 201.5 mm, vias 0 -> 1
- net GND: track 126.4 -> 78.1 mm
- net VCC: track 88.2 -> 48.4 mm, vias 1 -> 0
- net COL7: track 194.1 -> 160.9 mm
- net ROW3: track 175.2 -> 194.6 mm, vias 2 -> 0
- net COL0: track 174.7 -> 158.0 mm
- net COL4: track 122.3 -> 109.1 mm, vias 0 -> 1
- net Net-(D31-Pad2): track 38.7 -> 26.1 mm
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
Commit message: 4 encoders
Parts:
- added ec11-3: RotaryEncoder_Switch, Rotary_Encoder:RotaryEncoder_Alps_EC11E-Switch_Vertical_H20mm, F.Cu at (69.4, 107.4)
- added ec11-4: RotaryEncoder_Switch, Rotary_Encoder:RotaryEncoder_Alps_EC11E-Switch_Vertical_H20mm, F.Cu at (232.4, 112.0)
Connections:
- U1 pad 4: unconnected-(U1-Pad4) -> ENC2P1
- U1 pad 5: unconnected-(U1-Pad5) -> ENC2P2
- U1 pad 6: unconnected-(U1-Pad6) -> ENC3P1
- U1 pad 7: unconnected-(U1-Pad7) -> ENC3P2
Routing:
- net ENC3P1: track 0.00 -> 235.0 mm, vias 0 -> 3
- net GND: track 78.1 -> 291.7 mm, vias 1 -> 3
- net ENC3P2: track 0.00 -> 181.1 mm, vias 0 -> 4
- net ENC2P1: track 0.00 -> 161.8 mm, vias 0 -> 1
- net ENC2P2: track 0.00 -> 148.2 mm, vias 0 -> 3
- net ROW3: track 194.6 -> 255.5 mm, vias 0 -> 1
- net COL2: track 159.7 -> 172.4 mm
- net COL8: track 264.4 -> 271.0 mm
- net COL7: track 160.9 -> 164.0 mm
- net Net-(D36-Pad2): track 35.7 -> 36.2 mm
